Commit message: updated urdf to include ground contact link

File: ros2_ws/src/orion_description/urdf/orion.urdf (robot description, URDF)
Before this commit: robot orion, 7 links, 6 joints
Links:
- added link base_footprint
- link imu_link: mass 1e-9 -> None
Joints:
- added joint base_footprint_joint: type fixed, parent base_footprint, child base_link, origin xyz=0 0 0.0418 rpy=0 0 0
- joint base_yaw_joint: axis 0 0 1 -> 0.999999999987 3.67320510325e-06 3.67320510333e-06; child base_link -> shoulder_mount_link; origin xyz=0.04111 7.30741e-16 -0.0192 rpy=-1.5708 5.39003e-15 1.5708 -> xyz=0 0 0 rpy=-2.3561944902 1.5707911321 2.3561944902; parent shoulder_mount_link -> base_link
- joint elbow_pitch_joint: origin xyz=0.105806 -0.0129789 0.301237 rpy=1.5708 -1.54809 -0.308645 -> xyz=0.09997366 -0.0312716 0.218327 rpy=1.5708 -1.54809 -0.308645
- joint imu_fixed_joint: axis 0 0 0 -> (none)
- joint shoulder_pitch_joint: axis 0 0 1 -> -0.3037692089 -0.952745646919 1.11580660844e-06; child shoulder_mount_link -> upper_arm_link; origin xyz=0.00583234 0.0182927 0.08291 rpy=-1.26215 1.5708 0 -> xyz=-0.04111 0 0.0192 rpy=1.57079749794 -0.308646326793 -1.57080018218; parent upper_arm_link -> shoulder_mount_link

Commit message: added gezebo controll interfaces

File: ros2_ws/src/orion_description/urdf/orion.urdf (robot description, URDF)
Before this commit: robot orion, 8 links, 7 joints
Links:
- link base_link: geometry collision mesh filename=package://orion_description/meshes/ge_27.stl; collision mesh filename=package://orion_description/meshes/lamp_base.stl
- link forearm_link: geometry collision mesh filename=package://orion_description/meshes/ge_27.stl; collision mesh filename=package://orion_description/meshes/lamparm__elbow_wrist.stl
- link head_roll_link: geometry collision mesh filename=package://orion_description/meshes/ge_27.stl; collision mesh filename=package://orion_description/meshes/lamparm__wrist_head.stl
- link shoulder_mount_link: geometry collision mesh filename=package://orion_description/meshes/ge_27.stl; collision mesh filename=package://orion_description/meshes/lamparm__wrist_head.stl
- link upper_arm_link: geometry collision mesh filename=package://orion_description/meshes/ge_27.stl; collision mesh filename=package://orion_description/meshes/lamparm__base_elbow.stl

Commit message: checkpoint

File: ros2_ws/src/orion_description/urdf/orion.urdf (robot description, URDF)
Before this commit: robot orion, 8 links, 7 joints
Links:
- link base_link: geometry collision box size=0.225084 0.205614 0.04; collision mesh filename=package://orion_description/meshes/ge_27.stl

Commit message: updated limits for shoulder pitch

File: ros2_ws/src/orion_description/urdf/orion.urdf (robot description, URDF)
Before this commit: robot orion, 8 links, 7 joints
Joints:
- joint shoulder_pitch_joint: limit lower=-1.08426 upper=2.05734 effort=10 velocity=10 -> lower=-1.33456 upper=2.05734 effort=10 velocity=10

Commit message: motion updates

File: ros2_ws/src/orion_description/urdf/orion.urdf (robot description, URDF)
Before this commit: robot orion, 8 links, 7 joints
Joints:
- joint elbow_pitch_joint: limit lower=-2.82002 upper=0.321569 effort=10 velocity=10 -> lower=-2.82002 upper=0.76699 effort=10 velocity=10
