Commit message: multi lamp pairing + pairing simplification + v2 home update

File: description/urdf/orion-v2.urdf (robot description, URDF)
Before this commit: robot orion_v2, 6 links, 5 joints
Joints:
- joint base_yaw_joint: axis 0 0 1 -> 0 0 -1
- joint head_roll_joint: axis 0 0 1 -> 0 0 -1

Commit message: camera P1: add URDF-derived camera and light kinematics
Add nominal fixed camera_optical_frame and light_frame mounts to the V2
URDF and matching MuJoCo camera/site definitions. Preserve existing model
links, joint origins, axes, ranges and meshes. Document ROS optical axes
(+X right, +Y down, +Z forward) and MuJoCo's camera-axis conversion.

Add Kinematics::from_urdf and fallible fk(&JointPositions), returning camera
and light poses in the base frame. Read origins and axes from a validated
connected URDF tree; load once outside the control tick. FK rejects wrong
joint names and non-finite angles, does no I/O or allocation on valid input,
and does not treat CAD limits as servo calibration. Add the user-approved
roxmltree 0.21.1 dependency and update runtime/coordinator lockfiles.

Commit independently generated MuJoCo fixtures for zero, home, left/right
looks and 20 seeded poses inside model limits, with source hashes and a
reproducible generator. Test full poses within 1 mm and 0.5 degrees, home
position/upward view, yaw/pitch signs, transform ordering, invalid inputs,
and URDF tree validation. Document the API and fixture procedure.

Checks:
- cargo fmt --manifest-path runtime/Cargo.toml --check: passed.
- cargo test --manifest-path runtime/Cargo.toml --all-targets --locked:
  265 passed. Initial sandbox run denied three Unix socket binds;
  unchanged suite passed with local socket permission.
- cargo build --manifest-path runtime/Cargo.toml --bins --locked: passed.
- .venv/bin/python -m unittest discover -s runtime/tests -p 'test_*.py' -v:
  35 passed, using the existing MuJoCo environment and local socket permission.
- python3 -m unittest discover -s tests -p 'test_*.py' -v: 3 passed.
- .venv/bin/python -m pytest tests/test_robot_description.py
  simulation/mujoco/test_v2_model.py -q: 12 passed, 2 subtests passed.
- .venv/bin/python tests/generate_camera_fk_fixtures.py --check:
  all 24 fixture poses reproduce with MuJoCo 3.10.0.
- cargo check --manifest-path coordinator/Cargo.toml --locked: passed.
- New URDF/MJCF mount tests fail against the original models, as required.
- Model structure comparison after removing new mounts: existing structure
  unchanged. Description README file links resolve. git diff --check: passed.

Unverified on hardware: fitted camera/light mount offsets, camera-to-head
rotation correction, lens intrinsics, and physical light-beam alignment.
P1 validates nominal CAD geometry only; no lamp hardware check was run.

File: description/urdf/orion-v2.urdf (robot description, URDF)
Before this commit: robot orion_v2, 6 links, 5 joints
Links:
- added link camera_optical_frame
- added link light_frame
Joints:
- added joint camera_optical_joint: type fixed, parent v21_neck_swivel_link, child camera_optical_frame, origin xyz=0 -0.082 0.0157 rpy=-1.5707963267948966 0 3.141592653589793
- added joint light_joint: type fixed, parent v21_neck_swivel_link, child light_frame, origin xyz=0 -0.077 0.020 rpy=-1.5707963267948966 0 3.141592653589793

Commit message: camera P4: V2 URDF zero matches the robot
Bake the exact measured pitch references into V2 URDF origins and MJCF refs.
Use safe calibrated ranges in both models and record the calibration hash
and applied model paths. Remove only V2 Studio preview offsets; keep V1.
Regenerate camera/light FK fixtures and document the bent calibrated zero.

Prove old FK(q - ref) equals new FK(q) to 1e-12 at home, rest and random
poses; verify the measured home link/view angles and every V2 pose limit.
Update sign tests for the baked geometry while retaining direction checks.
No servo calibration, existing pose/motion/scene or mesh changes.

Checks (all pass):
- cargo fmt --manifest-path runtime/Cargo.toml --check
- cargo test --manifest-path runtime/Cargo.toml --all-targets --locked
  (270 library tests plus 1 trajectory CLI test; native MuJoCo included)
- cargo test --manifest-path runtime/Cargo.toml --doc --locked
- cargo build --manifest-path runtime/Cargo.toml --locked
- python3 -m unittest discover -s runtime/tests -p 'test_*.py' -v (37)
- python3 -m unittest discover -s tests -p 'test_*.py' -v (4)
- python3 -m unittest discover -s orion_studio/tests -v (71)
- pnpm --dir orion_studio test (287), pnpm --dir orion_studio build
  (PATH selects installed Node 22.13.1; existing chunk-size warning)
- .venv/bin/python -m pytest tests/test_robot_description.py
  simulation/mujoco/test_v2_model.py (13)
- .venv/bin/python tests/generate_camera_fk_fixtures.py --check (24 poses)
- git diff --check
Socket suites rerun with local socket access after sandbox denial.

Hardware unverified: compare the home preview to the assembled lamp;
calibration and measured camera mount/intrinsics remain physical evidence,
not a collision, balance or motor-tracking safety certification.

File: description/urdf/orion-v2.urdf (robot description, URDF)
Before this commit: robot orion_v2, 8 links, 7 joints
Joints:
- joint base_yaw_joint: limit lower=-1.5707963267948966 upper=1.5707963267948966 effort=0 velocity=0 -> lower=-1.4388739790367313 upper=1.5401167110371838 effort=0 velocity=0
- joint elbow_pitch_joint: limit lower=-2.705260340591211 upper=2.705260340591211 effort=0 velocity=0 -> lower=-1.5707963267948966 upper=1.069184609156292 effort=0 velocity=0; origin xyz=0.0 0.0 0.15000000000000002 rpy=0 0 0 -> xyz=0.0 0.0 0.15000000000000002 rpy=1.5 0 0
- joint head_pitch_joint: limit lower=-1.5707963267948966 upper=1.5707963267948966 effort=0 velocity=0 -> lower=-0.6718835850939109 upper=1.3453011509757073 effort=0 velocity=0; origin xyz=0.0 0.0 0.131 rpy=0 0 0 -> xyz=0.0 0.0 0.131 rpy=-0.07 0 0
- joint head_roll_joint: limit lower=-1.5707963267948966 upper=1.5707963267948966 effort=0 velocity=0 -> lower=-1.7778837331594581 upper=1.6122138080678088 effort=0 velocity=0
- joint shoulder_pitch_joint: limit lower=-1.5707963267948966 upper=1.5707963267948966 effort=0 velocity=0 -> lower=-0.5553010452146021 upper=1.2547962844904545 effort=0 velocity=0; origin xyz=0.0 0.0 0.05299999999999999 rpy=0 0 0 -> xyz=0.0 0.0 0.05299999999999999 rpy=-1.118 0 0

Commit message: Use V2 mechanical rest zero and ship Raspberry Pi OS releases

File: description/urdf/orion-v2.urdf (robot description, URDF)
Before this commit: robot orion_v2, 8 links, 7 joints
Joints:
- joint base_yaw_joint: limit lower=-1.4388739790367313 upper=1.5401167110371838 effort=0 velocity=0 -> lower=-1.4879613642490719 upper=1.4910293258248433 effort=0 velocity=0; origin xyz=0.0 0.0 0.060000000000000005 rpy=0 0 0 -> xyz=0.0 0.0 0.060000000000000005 rpy=0.0 0.0 -0.04908738521234052
- joint elbow_pitch_joint: limit lower=-1.5707963267948966 upper=1.069184609156292 effort=0 velocity=0 -> lower=-2.45283527982914 upper=0.18714565612204836 effort=0 velocity=0; origin xyz=0.0 0.0 0.15000000000000002 rpy=1.5 0 0 -> xyz=0.0 0.0 0.15000000000000002 rpy=2.297002562636047 0.0 0.0
- joint head_pitch_joint: limit lower=-0.6718835850939109 upper=1.3453011509757073 effort=0 velocity=0 -> lower=-0.8912428377615575 upper=1.1259418983080607 effort=0 velocity=0; origin xyz=0.0 0.0 0.131 rpy=-0.07 0 0 -> xyz=0.0 0.0 0.131 rpy=0.08911356580737373 0.0 0.0
- joint head_roll_joint: limit lower=-1.7778837331594581 upper=1.6122138080678088 effort=0 velocity=0 -> lower=-1.7640779060684875 upper=1.6260196351587795 effort=0 velocity=0; origin xyz=0.0 -0.0175 0.04899999999999999 rpy=0 0 0 -> xyz=0.0 -0.0175 0.04899999999999999 rpy=-0.0 -0.0 0.01380582709097077
- joint shoulder_pitch_joint: limit lower=-0.5553010452146021 upper=1.2547962844904545 effort=0 velocity=0 -> lower=0.0 upper=1.8100973297050567 effort=0 velocity=0; origin xyz=0.0 0.0 0.05299999999999999 rpy=-1.118 0 0 -> xyz=0.0 0.0 0.05299999999999999 rpy=-1.5980932991569734 -0.0 -0.0
